Commit message: Enable hardware interface compilation

File: modelidar/urdf/ros2_control.xacro (robot description, xacro)
@@ -2,24 +2,25 @@
 <robot xmlns:xacro="http://www.ros.org/wiki/xacro">
  <xacro:macro name="modelidar_ros2_control" params="name prefix use_mock_hardware">
+<!-- <parameters>$(find articubot_one)/config/my_controllers.yaml</parameters> -->
 <ros2_control name="${name}" type="system">
       <xacro:unless value="${use_mock_hardware}">
         <hardware>
-          <plugin>modelidar/ModelidarystemHardware</plugin>
+          <plugin>modelidar/ModelidarSystemHardware</plugin>
           <param name="example_param_hw_start_duration_sec">0</param>
           <param name="example_param_hw_stop_duration_sec">3.0</param>
         </hardware>
       </xacro:unless>
-      <xacro:if value="${use_mock_hardware}">
+      <!-- <xacro:if value="${use_mock_hardware}">
         <hardware>
           <plugin>mock_components/GenericSystem</plugin>
           <param name="calculate_dynamics">true</param>
         </hardware>
-      </xacro:if>
-      <joint name="${prefix}left_wheel_joint">
+      </xacro:if> -->
+      <joint name="${prefix}virtual_left_wheel_joint">
         <command_interface name="velocity"/>
         <state_interface name="position"/>
         <state_interface name="velocity"/>
       </joint>
-      <joint name="${prefix}right_wheel_joint">
+      <joint name="${prefix}virtual_right_wheel_joint">
         <command_interface name="velocity"/>
         <state_interface name="position"/>

File: modelidar/urdf/wild_thumper.urdf.xacro (robot description, xacro)
@@ -4,4 +4,6 @@
   	<xacro:arg name="use_mock_hardware" default="false" />
 	<xacro:property name="PI" value="3.1415926535897931" />
+	<xacro:property name="wheelbase" value="0.24" />
+	<xacro:property name="wheel_radius" value="0.05" />
 	<!-- Import Rviz colors -->
 	<xacro:include filename="materials.xacro" />
@@ -155,6 +157,4 @@
 		</joint>
 	</xacro:macro>
-	<xacro:property name="wheelbase" value="0.24" />
-	<xacro:property name="wheel_radius" value="0.05" />
 	<xacro:wheel prefix="$(arg prefix)" pos="rear" side="left"   xyz="-0.07525  +${wheelbase/2} -0.025" rpy="${-5*PI/180} 0 0" /> <!-- rear_left_wheel -->
 	<xacro:wheel prefix="$(arg prefix)" pos="rear" side="right"  xyz="-0.07525 -${wheelbase/2} -0.025" rpy="${5*PI/180} 0 0" /> <!-- rear_right_wheel -->

Commit message: Modelidar comms integrated in ros control Hardware Interface

File: modelidar/urdf/ros2_control.xacro (robot description, xacro)
@@ -9,4 +9,9 @@
           <param name="example_param_hw_start_duration_sec">0</param>
           <param name="example_param_hw_stop_duration_sec">3.0</param>
+          <param name="loop_rate">30</param>
+          <param name="device">/dev/ttyACM0</param>
+          <param name="baud_rate">115200</param>
+          <param name="timeout">1000</param>
+          <param name="enc_counts_per_rev">544</param> <!-- 16x34 for encoder DAGU RS003-Enco -->
         </hardware>
       </xacro:unless>

File: modelidar/urdf/wild_thumper.urdf.xacro (robot description, xacro)
@@ -6,4 +6,5 @@
 	<xacro:property name="wheelbase" value="0.24" />
 	<xacro:property name="wheel_radius" value="0.05" />
+	<xacro:property name="base_link_z" value="0.082" />
 	<!-- Import Rviz colors -->
 	<xacro:include filename="materials.xacro" />
@@ -75,10 +76,10 @@
 		<parent link="$(arg prefix)base_footprint"/>
 		<child link="$(arg prefix)base_link"/>
-		<origin xyz="0.0 0.0 0.082" rpy="0 0 0"/>
+		<origin xyz="0.0 0.0 ${base_link_z}" rpy="0 0 0"/>
 	</joint>
 	<joint name="$(arg prefix)mounting_plate_joint" type="fixed">
 		<parent link="$(arg prefix)base_link"/>
 		<child link="$(arg prefix)mounting_plate"/>
-		<origin xyz="0.0 0.0 0.044" rpy="0 0 0"/>
+		<origin xyz="0.0 0.0 ${0.044+0.03}" rpy="0 0 0"/>
 	</joint>
 	<joint name="$(arg prefix)imu_joint" type="fixed">
@@ -149,5 +150,5 @@
 		</link>
 		<joint name="${prefix}virtual_${side}_wheel_joint" type="continuous">
-		<parent link="${prefix}base_footprint"/>
+		<parent link="${prefix}base_link"/>
 		<child link="${ prefix}virtual_${side}_wheel"/>
 		<origin xyz="${xyz}" rpy="0 0 0"/>
@@ -161,6 +162,6 @@
 	<xacro:wheel prefix="$(arg prefix)" pos="front" side="left"  xyz=" 0.07525  +${wheelbase/2} -0.025" rpy="${-5*PI/180} 0 0" /> <!-- front_left_wheel -->
 	<xacro:wheel prefix="$(arg prefix)" pos="front" side="right" xyz=" 0.07525 -${wheelbase/2} -0.025" rpy="${5*PI/180} 0 0" /> <!-- front_right_wheel -->
-	<xacro:virtual_wheel prefix="$(arg prefix)" side="left" xyz="0 +${wheelbase/2} ${wheel_radius}"/> <!-- virtual_left_wheel -->
-	<xacro:virtual_wheel prefix="$(arg prefix)" side="right" xyz="0 -${wheelbase/2} ${wheel_radius}"/> <!-- virtual_right_wheel -->
+	<xacro:virtual_wheel prefix="$(arg prefix)" side="left" xyz="0 +${wheelbase/2} ${wheel_radius-base_link_z}"/> <!-- virtual_left_wheel -->
+	<xacro:virtual_wheel prefix="$(arg prefix)" side="right" xyz="0 -${wheelbase/2} ${wheel_radius-base_link_z}"/> <!-- virtual_right_wheel -->
 	<gazebo>
 		<plugin name="$(arg prefix)gazebo_ros_control" filename="libgazebo_ros_control.so">

Commit message: Fix close loop control for correct Odom TF

File: modelidar/urdf/ros2_control.xacro (robot description, xacro)
@@ -16,10 +16,10 @@
         </hardware>
       </xacro:unless>
-      <!-- <xacro:if value="${use_mock_hardware}">
+      <xacro:if value="${use_mock_hardware}">
         <hardware>
           <plugin>mock_components/GenericSystem</plugin>
           <param name="calculate_dynamics">true</param>
         </hardware>
-      </xacro:if> -->
+      </xacro:if>
       <joint name="${prefix}virtual_left_wheel_joint">
         <command_interface name="velocity"/>

File: modelidar/urdf/wild_thumper.urdf.xacro (robot description, xacro)
@@ -81,5 +81,5 @@
 		<parent link="$(arg prefix)base_link"/>
 		<child link="$(arg prefix)mounting_plate"/>
-		<origin xyz="0.0 0.0 ${0.044+0.03}" rpy="0 0 0"/>
+		<origin xyz="0.0 0.0 ${0.044+0.02}" rpy="0 0 0"/>
 	</joint>
 	<joint name="$(arg prefix)imu_joint" type="fixed">
